File: embedded/prototype-B/board-design/retrolight-main/retrolight-main.kicad_sch (KiCad schematic)
At the start: 43 parts, among them J1 Conn_02x03_Odd_Even, U1 TLC59108xPW, U2 TLC59108xPW

Commit message: [Refactored PCB design]
Renewed PCB design for the retrolight app.

Signed-off-by: Nicolae-Andrei Vasile <vasilenicolaeandrei@gmail.com>
Parts:
- removed C3: 10uF/6.3V/20%/C0603, Capacitor_SMD:C_0603_1608Metric_Pad1.08x0.95mm_HandSolder, symbol Device:C
- removed C4: 100nF/6.3V/20%/C0603, Capacitor_SMD:C_0603_1608Metric_Pad1.08x0.95mm_HandSolder, symbol Device:C
- removed D10, D11, D12, D13, D14, D15, D16, D9: LED, LED:LED_0505_1313Metric, symbol SparkFun-LED:LED
- removed R10, R11, R12, R13: 10K/R0603(NC), Resistor_SMD:R_0603_1608Metric_Pad0.98x0.95mm_HandSolder, symbol Device:R
- removed R14, R15, R16, R17: 0R/R0603, Resistor_SMD:R_0603_1608Metric_Pad0.98x0.95mm_HandSolder, symbol Device:R
- removed R18: 375R/R0603, Resistor_SMD:R_0603_1608Metric_Pad0.98x0.95mm_HandSolder, symbol Device:R
- removed U2: TLC59108xPW, Package_SO:TSSOP-20_4.4x6.5mm_P0.65mm, symbol Driver_LED:TLC59108xPW
- added R1, R2, R3, R4, R5, R6, R7, R8: 0R/R0603, Resistor_SMD:R_0603_1608Metric_Pad0.98x0.95mm_HandSolder, symbol Device:R
- H1, H2: footprint MountingHole:MountingHole_3.2mm_M3 -> MountingHole:MountingHole_2.2mm_M2_ISO7380
- renumbered R2 to R10, R3 to R11, R4 to R12, R5 to R13, R6 to R14, R7 to R15, R8 to R16, R9 to R17, R1 to R9
Connections:
- net VLED: now also R1.2, R2.2, R3.2, R4.2, R5.2, R6.2, R7.2, R8.2; no longer D1.2 (A), D2.2 (A), D3.2 (A), D4.2 (A), D5.2 (A), D6.2 (A), D7.2 (A), D8.2 (A)
- new net: D4.2 (A), R4.1
- new net: D1.2 (A), R1.1
- new net: D7.2 (A), R7.1
- new net: D3.2 (A), R3.1
- new net: D2.2 (A), R2.1
- new net: D8.2 (A), R8.1
- new net: D5.2 (A), R5.1
- new net: D6.2 (A), R6.1
Other:
- title: (none) -> Retrolight
- moved on the sheet: C1, C2, D1, H1, J1, R10, R11, R12, R13, R14, R15, R16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

Commit message: [Light] Rework
Refactored light module design to match the newest changes for the
central unit.

Signed-off-by: Nicolae-Andrei Prodan <vasilenicolaeandrei@gmail.com>
Parts:
- removed D1, D2, D3, D4, D5, D6, D7, D8: LED, LED:LED_0505_1313Metric, symbol SparkFun-LED:LED
- removed H1, H2: MountingHole, MountingHole:MountingHole_2.2mm_M2_ISO7380, symbol Mechanical:MountingHole
- removed J1: Conn_02x03_Odd_Even, Connector_PinSocket_2.54mm:PinSocket_2x03_P2.54mm_Vertical, symbol Connector_Generic:Conn_02x03_Odd_Even
- added D1, D2, D3, D4, D5, D6, D7, D8: LED, LED:LED_0505_1313Metric, symbol Device:LED
- added D9: MBRS130LT3G, Diode_SMD:D_SMB, symbol Device:D_Schottky
- added H1, H2: MountingHole_Pad, MountingHole:MountingHole_4.3mm_M4_ISO7380_Pad, symbol Mechanical:MountingHole_Pad
- added J1: Conn_02x05_Odd_Even, Connector_IDC:IDC-Header_2x05_P2.54mm_Vertical, symbol Connector_Generic:Conn_02x05_Odd_Even
- renumbered R9 to R1, R1 to R10, R2 to R11, R3 to R12, R4 to R13, R5 to R14, R6 to R15, R7 to R16, R8 to R17, R13 to R2, R10 to R3, R14 to R4, R11 to R5, R15 to R6, R12 to R7, R16 to R8, R17 to R9
Connections:
- net VLED is gone; now on net VCC: R10.2, R11.2, R12.2, R13.2, R14.2, R15.2, R16.2, R17.2
- net GND: now also H1.1, H2.1, J1.10 (Pin_10)
- net SCL: now also J1.5 (Pin_5)
- net SDA: now also J1.3 (Pin_3)
- net VCC: now also D9.1 (K)
- net ~{RESET}: now also J1.7 (Pin_7)
- net at R13.1: now also D4.2 (A)
- net at U1.6 (~{OUT0}): now also D1.1 (K)
- net at R10.1: now also D1.2 (A)
- net at U1.10 (~{OUT3}): now also D4.1 (K)
- net at R16.1: now also D7.2 (A)
- net at U1.11 (~{OUT4}): now also D5.1 (K)
- net at U1.12 (~{OUT5}): now also D6.1 (K)
- net at U1.14 (~{OUT6}): now also D7.1 (K)
- net at U1.15 (~{OUT7}): now also D8.1 (K)
- net at U1.7 (~{OUT1}): now also D2.1 (K)
- net at U1.9 (~{OUT2}): now also D3.1 (K)
- net at R12.1: now also D3.2 (A)
- net at R11.1: now also D2.2 (A)
- net at R17.1: now also D8.2 (A)
- net at R14.1: now also D5.2 (A)
- net at R15.1: now also D6.2 (A)
- new net: D9.2 (A), J1.1 (Pin_1)
- no-connect marks 0 -> 5
